File: rc522.kicad_sch (KiCad schematic)
At the start: 21 parts, among them U1 MFRC52202HN1,151, Y1 27.12 MHz Crystal

Commit message: PCB: one layout done, trying replication now
Parts:
- C1, C10, C11, C12, C13, C14, C2, C3, C4, C5, C6, C7, C8, C9: footprint (none) -> Capacitor_SMD:C_0603_1608Metric
- L1, L2: footprint (none) -> Inductor_SMD:L_0603_1608Metric
- R1, R2, R3: footprint (none) -> Resistor_SMD:R_0603_1608Metric
- Y1: footprint (none) -> Crystal:Crystal_SMD_3225-4Pin_3.2x2.5mm
Connections:
- net GND: no longer C10.1, C11.1, C12.2, C6.2, C7.2, C8.2, C9.2
- new net: C11.1, C12.2, C8.2
- new net: C10.1, C6.2, C7.2, C9.2
Changed lines of the file:
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@@
 	)
 	(junction
-		(at 247.65 106.68)
-		(diameter 0)
-		(color 0 0 0 0)
-	)
-	(junction
 		(at 31.75 87.63)
 		(diameter 0)
@@
 	(wire
 		(pts
-			(xy 247.65 99.06) (xy 247.65 106.68)
-		)
-		(stroke
-			(width 0)
-			(type default)
-		)
-	)
-	(wire
-		(pts
 			(xy 86.36 123.19) (xy 86.36 134.62)
 		)
@@
 	(wire
 		(pts
-			(xy 247.65 106.68) (xy 247.65 114.3)
-		)
-		(stroke
-			(width 0)
-			(type default)
-		)
-	)
-	(wire
-		(pts
 			(xy 139.7 91.44) (xy 144.78 91.44)
 		)
@@
 			)
 		)
-		(property "Footprint" ""
+		(property "Footprint" "Capacitor_SMD:C_0603_1608Metric"
 			(at 231.14 110.49 0)
 			(hide yes)
@@
 			)
 		)
-		(property "Footprint" ""
+		(property "Footprint" "Capacitor_SMD:C_0603_1608Metric"
 			(at 215.9 102.87 0)
 			(hide yes)
@@
 			)
 		)
-		(property "Footprint" ""
+		(property "Footprint" "Capacitor_SMD:C_0603_1608Metric"
 			(at 231.14 102.87 0)
 			(hide yes)
@@
 			)
 		)
-		(property "Footprint" ""
+		(property "Footprint" "Capacitor_SMD:C_0603_1608Metric"
 			(at 78.74 137.16 0)
 			(hide yes)
@@
 			)
 		)
-		(property "Footprint" ""
+		(property "Footprint" "Capacitor_SMD:C_0603_1608Metric"
 			(at 186.69 110.49 0)
 			(hide yes)
@@
 			)
 		)
-		(property "Footprint" ""
+		(property "Footprint" "Resistor_SMD:R_0603_1608Metric"
 			(at 41.91 100.33 0)
 			(hide yes)
@@
 			)
 		)
-		(property "Footprint" ""
+		(property "Footprint" "Capacitor_SMD:C_0603_1608Metric"
 			(at 201.93 114.3 0)
 			(hide yes)
@@
 			)
 		)
-		(property "Footprint" ""
+		(property "Footprint" "Capacitor_SMD:C_0603_1608Metric"
 			(at 97.79 128.27 0)
 			(hide yes)
@@
 			)
 		)
-		(property "Footprint" ""
+		(property "Footprint" "Crystal:Crystal_SMD_3225-4Pin_3.2x2.5mm"
 			(at 137.16 91.44 0)
 			(hide yes)
@@
 			)
 		)
-		(property "Footprint" ""
+		(property "Footprint" "Capacitor_SMD:C_0603_1608Metric"
 			(at 186.69 102.87 0)
 			(hide yes)
@@
 			)
 		)
-		(property "Footprint" ""
+		(property "Footprint" "Capacitor_SMD:C_0603_1608Metric"
 			(at 140.97 99.06 0)
 			(hide yes)
@@
 			)
 		)
-		(property "Footprint" ""
+		(property "Footprint" "Inductor_SMD:L_0603_1608Metric"
 			(at 180.34 114.3 0)
 			(hide yes)
@@
 			)
 		)
-		(property "Footprint" ""
+		(property "Footprint" "Inductor_SMD:L_0603_1608Metric"
 			(at 180.34 99.06 0)
 			(hide yes)
@@
 			)
 		)
-		(property "Footprint" ""
+		(property "Footprint" "Capacitor_SMD:C_0603_1608Metric"
 			(at 205.74 90.17 0)
 			(hide yes)
@@
 			)
 		)
-		(property "Footprint" ""
+		(property "Footprint" "Capacitor_SMD:C_0603_1608Metric"
 			(at 201.93 99.06 0)
 			(hide yes)
@@
 			)
 		)
-		(property "Footprint" ""
+		(property "Footprint" "Capacitor_SMD:C_0603_1608Metric"
 			(at 140.97 85.09 0)
 			(hide yes)
@@
 			)
 		)
-		(property "Footprint" ""
+		(property "Footprint" "Resistor_SMD:R_0603_1608Metric"
 			(at 181.61 85.09 0)
 			(hide yes)
@@
 			)
 		)
-		(property "Footprint" ""
+		(property "Footprint" "Capacitor_SMD:C_0603_1608Metric"
 			(at 215.9 110.49 0)
 			(hide yes)
@@
 			)
 		)
-		(property "Footprint" ""
+		(property "Footprint" "Resistor_SMD:R_0603_1608Metric"
 			(at 193.04 90.17 0)
 			(hide yes)
@@
 			)
 		)
-		(property "Footprint" ""
+		(property "Footprint" "Capacitor_SMD:C_0603_1608Metric"
 			(at 31.75 82.55 0)
 			(hide yes)

Commit message: Previous stuff and im now at a point where a single reader circuit should be ready for replecation
Parts:
- removed C14: 100nF, Capacitor_SMD:C_0603_1608Metric, symbol Device:C_Small
- added C58, C62: 100nF, Capacitor_SMD:C_0603_1608Metric, symbol Device:C_Small
- added C66: 1uF, Capacitor_SMD:C_0603_1608Metric, symbol Device:C_Small
- added R13: 10k, Resistor_SMD:R_0603_1608Metric, symbol Device:R_Small
- added TP1: Antenna, symbol Connector:TestPoint_2Pole
Connections:
- net +3V3: now also C58.1, C62.1, C66.1, R13.1
- net GND: now also C58.2, C62.2, C66.2
- net MFSDA-CS: now also R13.2
- net at C11.1, C12.2, C8.2: now also C10.1, C6.2, C7.2, C9.2, TP1.1, TP1.2
Other:
- moved on the sheet: C13

Commit message: added BOMs and Plot
Parts:
- C1, C2: value 15pF -> 15pF NP0; DigiKey PN (none) -> 1276-1296-2-ND; DigiKey URL (none) -> https://www.digikey.de/de/products/detail/samsung-electro-m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; LCSC Part (none) -> C1645
- C10, C12: value 10PF -> 10pF NP0; DigiKey PN (none) -> 1276-1027-2-ND; DigiKey URL (none) -> https://www.digikey.de/de/products/detail/samsung-electro-m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; LCSC Part (none) -> C1640
- C11, C9: value 180PF -> 180pF NP0; DigiKey PN (none) -> 490-1433-2-ND; DigiKey URL (none) -> https://www.digikey.de/de/products/detail/murata-electronic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; LCSC Part (none) -> C1683
- C13, C3, C58, C6, C62: DigiKey PN (none) -> 1276-1000-2-ND; DigiKey URL (none) -> https://www.digikey.de/de/products/detail/samsung-electro-m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; LCSC Part (none) -> C14663
- C4, C5: value 47PF -> 47pF NP0; DigiKey PN (none) -> 1276-1037-2-ND; DigiKey URL (none) -> https://www.digikey.de/de/products/detail/samsung-electro-m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; LCSC Part (none) -> C1665
- C66: DigiKey PN (none) -> 1276-1860-2-ND; DigiKey URL (none) -> https://www.digikey.de/de/products/detail/samsung-electro-m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; LCSC Part (none) -> C15849
- C7, C8: value 15PF -> 15pF NP0; DigiKey PN (none) -> 1276-1296-2-ND; DigiKey URL (none) -> https://www.digikey.de/de/products/detail/samsung-electro-m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; LCSC Part (none) -> C1645
- L1, L2: DigiKey PN (none) -> 445-6754-2-ND; DigiKey URL (none) -> https://www.digikey.de/de/products/detail/tdk/MLZ1608N2R2LT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; LCSC Part (none) -> C531282
- R1: DigiKey PN (none) -> 311-820HRTR-ND; DigiKey URL (none) -> https://www.digikey.de/de/products/detail/yageo/RC0603FR-07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; LCSC Part (none) -> C23179
- R13: DigiKey PN (none) -> 311-10.0KHRTR-ND; DigiKey URL (none) -> https://www.digikey.de/de/products/detail/yageo/RC0603FR-07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; LCSC Part (none) -> C25804
- R2: DigiKey PN (none) -> 311-5.10KHRTR-ND; DigiKey URL (none) -> https://www.digikey.de/de/products/detail/yageo/RC0603FR-07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; LCSC Part (none) -> C23186
- R3: value 10K -> 10k; DigiKey PN (none) -> 311-10.0KHRTR-ND; DigiKey URL (none) -> https://www.digikey.de/de/products/detail/yageo/RC0603FR-07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; LCSC Part (none) -> C25804
- TP1: Note (none) -> DNP; now not fitted; now left out of the parts list
- U1: Note (none) -> Aliexpress
- Y1: DigiKey PN (none) -> 2151-RH100-27.120-10-F-1010-TR-ND; DigiKey URL (none) -> https://www.digikey.de/de/products/detail/raltron-electroni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; LCSC Part (none) -> C29975
