File: sub-board.kicad_sch (KiCad schematic)
At the start: 6 parts, among them J1 IN1, J2 IN2, J3 OUT1, J4 OUT2, U2 SN74HC595N

Commit message: PCB: one layout done, trying replication now
Parts:
- C57: footprint (none) -> Capacitor_SMD:C_0603_1608Metric
- J1, J2: footprint (none) -> Connector_PinSocket_2.54mm:PinSocket_1x09_P2.54mm_Horizontal
- J3, J4: footprint (none) -> Connector_PinHeader_2.54mm:PinHeader_1x09_P2.54mm_Horizontal
Changed lines of the file:
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@@
 			)
 		)
-		(property "Footprint" ""
+		(property "Footprint" "Connector_PinSocket_2.54mm:PinSocket_1x09_P2.54mm_Horizontal"
 			(at 212.09 109.22 0)
 			(hide yes)
@@
 			)
 		)
-		(property "Footprint" ""
+		(property "Footprint" "Connector_PinHeader_2.54mm:PinHeader_1x09_P2.54mm_Horizontal"
 			(at 241.3 80.01 0)
 			(hide yes)
@@
 			)
 		)
-		(property "Footprint" ""
+		(property "Footprint" "Capacitor_SMD:C_0603_1608Metric"
 			(at 134.62 83.82 0)
 			(hide yes)
@@
 			)
 		)
-		(property "Footprint" ""
+		(property "Footprint" "Connector_PinSocket_2.54mm:PinSocket_1x09_P2.54mm_Horizontal"
 			(at 212.09 80.01 0)
 			(hide yes)
@@
 			)
 		)
-		(property "Footprint" ""
+		(property "Footprint" "Connector_PinHeader_2.54mm:PinHeader_1x09_P2.54mm_Horizontal"
 			(at 241.3 109.22 0)
 			(hide yes)

Commit message: Previous stuff and im now at a point where a single reader circuit should be ready for replecation
Parts:
- removed J1: IN1, Connector_PinSocket_2.54mm:PinSocket_1x09_P2.54mm_Horizontal, symbol Connector_Generic:Conn_01x09
- removed J2: IN2, Connector_PinSocket_2.54mm:PinSocket_1x09_P2.54mm_Horizontal, symbol Connector_Generic:Conn_01x09
- removed J3: OUT1, Connector_PinHeader_2.54mm:PinHeader_1x09_P2.54mm_Horizontal, symbol Connector_Generic:Conn_01x09
- removed J4: OUT2, Connector_PinHeader_2.54mm:PinHeader_1x09_P2.54mm_Horizontal, symbol Connector_Generic:Conn_01x09
- added J1: IN1, Connector_PinSocket_2.54mm:PinSocket_1x10_P2.54mm_Horizontal, symbol Connector_Generic:Conn_01x10
- added J2: OUT1, Connector_PinSocket_2.54mm:PinSocket_1x10_P2.54mm_Horizontal, symbol Connector_Generic:Conn_01x10
- added J3: IN2, Connector_PinSocket_2.54mm:PinSocket_1x10_P2.54mm_Horizontal, symbol Connector_Generic:Conn_01x10
- added J4: OUT2, Connector_PinSocket_2.54mm:PinSocket_1x10_P2.54mm_Horizontal, symbol Connector_Generic:Conn_01x10
Connections:
- net +3V3: now also J1.1 (Pin_1), J2.1 (Pin_1), J3.1 (Pin_1), J4.1 (Pin_1)
- net GND: now also J1.2 (Pin_2), J2.2 (Pin_2), J3.2 (Pin_2), J4.2 (Pin_2); no longer U2.13 (~{OE})
- net MISO: now also J1.4 (Pin_4), J2.4 (Pin_4), J3.4 (Pin_4), J4.4 (Pin_4)
- net MOSI: now also J1.3 (Pin_3), J2.3 (Pin_3), J3.3 (Pin_3), J4.3 (Pin_3)
- net RCLK: now also J1.9 (Pin_9), J2.9 (Pin_9), J3.9 (Pin_9), J4.9 (Pin_9)
- net RST: now also J1.6 (Pin_6), J2.6 (Pin_6), J3.6 (Pin_6), J4.6 (Pin_6)
- net SCK: now also J1.5 (Pin_5), J2.5 (Pin_5), J3.5 (Pin_5), J4.5 (Pin_5)
- net SER: now also J1.10 (Pin_10), J3.10 (Pin_10)
- net SER_OUT: now also J2.10 (Pin_10), J4.10 (Pin_10)
- net SRCLK: now also J1.8 (Pin_8), J2.8 (Pin_8), J3.8 (Pin_8), J4.8 (Pin_8)
- new net OE: J1.7 (Pin_7), J2.7 (Pin_7), J3.7 (Pin_7), J4.7 (Pin_7), U2.13 (~{OE})

Commit message: added BOMs and Plot
Parts:
- C57: DigiKey PN (none) -> 1276-1000-2-ND; DigiKey URL (none) -> https://www.digikey.de/de/products/detail/samsung-electro-m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; LCSC Part (none) -> C14663
- J1: value IN1 -> IN; Note (none) -> Generic
- J2: value OUT1 -> OUT; Note (none) -> Generic
- J3: value IN2 -> IN; Note (none) -> Generic
- J4: value OUT2 -> OUT; Note (none) -> Generic
- U2: DigiKey PN (none) -> 296-1600-5-ND; DigiKey URL (none) -> https://www.digikey.de/de/products/detail/texas-instruments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
